Commit message: Fixed relative paths

File: euroc_slam/urdf/firefly.urdf (robot description, URDF)
Before this commit: robot firefly, 8 links, 7 joints
Links:
- link firefly/base_link_inertia: geometry collision box size=0.1 0.1 0.16; visual mesh filename=meshes/firefly_purple.dae scale=1 1 1
- link firefly/rotor_0: geometry collision cylinder length=0.005 radius=0.1; visual mesh filename=meshes/propeller_ccw_purple.dae scale=0.1 0.1 0.1
- link firefly/rotor_1: geometry collision cylinder length=0.005 radius=0.1; visual mesh filename=meshes/propeller_cw_purple.dae scale=0.1 0.1 0.1
- link firefly/rotor_2: geometry collision cylinder length=0.005 radius=0.1; visual mesh filename=meshes/propeller_ccw_purple.dae scale=0.1 0.1 0.1
- link firefly/rotor_3: geometry collision cylinder length=0.005 radius=0.1; visual mesh filename=meshes/propeller_cw_purple.dae scale=0.1 0.1 0.1
- link firefly/rotor_4: geometry collision cylinder length=0.005 radius=0.1; visual mesh filename=meshes/propeller_ccw_purple.dae scale=0.1 0.1 0.1
- link firefly/rotor_5: geometry collision cylinder length=0.005 radius=0.1; visual mesh filename=meshes/propeller_cw_purple.dae scale=0.1 0.1 0.1

Commit message: changed pasths

File: euroc_slam/urdf/firefly.urdf (robot description, URDF)
Before this commit: robot firefly, 8 links, 7 joints
Links:
- link firefly/base_link_inertia: geometry collision box size=0.1 0.1 0.16; visual mesh filename=../meshes/firefly_purple.dae scale=1 1 1
- link firefly/rotor_0: geometry collision cylinder length=0.005 radius=0.1; visual mesh filename=../meshes/propeller_ccw_purple.dae scale=0.1 0.1 0.1
- link firefly/rotor_1: geometry collision cylinder length=0.005 radius=0.1; visual mesh filename=../meshes/propeller_cw_purple.dae scale=0.1 0.1 0.1
- link firefly/rotor_2: geometry collision cylinder length=0.005 radius=0.1; visual mesh filename=../meshes/propeller_ccw_purple.dae scale=0.1 0.1 0.1
- link firefly/rotor_3: geometry collision cylinder length=0.005 radius=0.1; visual mesh filename=../meshes/propeller_cw_purple.dae scale=0.1 0.1 0.1
- link firefly/rotor_4: geometry collision cylinder length=0.005 radius=0.1; visual mesh filename=../meshes/propeller_ccw_purple.dae scale=0.1 0.1 0.1
- link firefly/rotor_5: geometry collision cylinder length=0.005 radius=0.1; visual mesh filename=../meshes/propeller_cw_purple.dae scale=0.1 0.1 0.1
