Commit message: Made a seperate urdf for url viz

File: ros2_ws/src/euroc_slam/urdf/firefly_url.urdf (robot description, URDF)
Before this commit: robot firefly, 8 links, 7 joints
Links:
- removed link firefly_base_link
- removed link firefly_base_link_inertia
- removed link firefly_rotor_0
- removed link firefly_rotor_1
- removed link firefly_rotor_2
- removed link firefly_rotor_3
- removed link firefly_rotor_4
- removed link firefly_rotor_5
- added link firefly/base_link
- added link firefly/base_link_inertia, mass 1.5; collision box size=0.1 0.1 0.16; visual mesh filename=package://euroc_slam/meshes/firefly_purple.dae scale=1 1 1
- added link firefly/rotor_0, mass 0.005; collision cylinder length=0.005 radius=0.1; visual mesh filename=package://euroc_slam/meshes/propeller_ccw_purple.dae scale=0.1 0.1 0.1
- added link firefly/rotor_1, mass 0.005; collision cylinder length=0.005 radius=0.1; visual mesh filename=package://euroc_slam/meshes/propeller_cw_purple.dae scale=0.1 0.1 0.1
- added link firefly/rotor_2, mass 0.005; collision cylinder length=0.005 radius=0.1; visual mesh filename=package://euroc_slam/meshes/propeller_ccw_purple.dae scale=0.1 0.1 0.1
- added link firefly/rotor_3, mass 0.005; collision cylinder length=0.005 radius=0.1; visual mesh filename=package://euroc_slam/meshes/propeller_cw_purple.dae scale=0.1 0.1 0.1
- added link firefly/rotor_4, mass 0.005; collision cylinder length=0.005 radius=0.1; visual mesh filename=package://euroc_slam/meshes/propeller_ccw_purple.dae scale=0.1 0.1 0.1
- added link firefly/rotor_5, mass 0.005; collision cylinder length=0.005 radius=0.1; visual mesh filename=package://euroc_slam/meshes/propeller_cw_purple.dae scale=0.1 0.1 0.1
Joints:
- removed joint firefly_base_joint
- removed joint firefly_rotor_0_joint
- removed joint firefly_rotor_1_joint
- removed joint firefly_rotor_2_joint
- removed joint firefly_rotor_3_joint
- removed joint firefly_rotor_4_joint
- removed joint firefly_rotor_5_joint
- added joint firefly/base_joint: type fixed, parent firefly/base_link, child firefly/base_link_inertia, origin xyz=0 0 0 rpy=0 0 0
- added joint firefly/rotor_0_joint: type continuous, parent firefly/base_link, child firefly/rotor_0, origin xyz=0.18619546181355998 0.1075 0.037 rpy=0 0 0, axis 0 0 1
- added joint firefly/rotor_1_joint: type continuous, parent firefly/base_link, child firefly/rotor_1, origin xyz=0 0.215 0.037 rpy=0 0 0, axis 0 0 1
- added joint firefly/rotor_2_joint: type continuous, parent firefly/base_link, child firefly/rotor_2, origin xyz=-0.18619546181355998 0.1075 0.037 rpy=0 0 0, axis 0 0 1
- added joint firefly/rotor_3_joint: type continuous, parent firefly/base_link, child firefly/rotor_3, origin xyz=-0.18619546181355998 -0.1075 0.037 rpy=0 0 0, axis 0 0 1
- added joint firefly/rotor_4_joint: type continuous, parent firefly/base_link, child firefly/rotor_4, origin xyz=0 -0.215 0.037 rpy=0 0 0, axis 0 0 1
- added joint firefly/rotor_5_joint: type continuous, parent firefly/base_link, child firefly/rotor_5, origin xyz=0.18619546181355998 -0.1075 0.037 rpy=0 0 0, axis 0 0 1
